File: pcb/pollin-lcd.kicad_pcb (KiCad board)
At the start: 2 copper layers, 248 x 56 mm, 18 parts, among them J1 Raspberry_Pi_2_3, J3 505110-4091, U1 TLV62568DBV

Commit message: things
Parts:
- removed ?: , clipboard:8f9f653c-d1d4-44ae-8881-cd5268ffe7a2
Connections:
- net /B0 renamed /Display connector/B0
- net /B1 renamed /Display connector/B1
- net /B2 renamed /Display connector/B2
- net /B3 renamed /Display connector/B3
- net /B4 renamed /Display connector/B4
- net /B5 renamed /Display connector/B5
- net /DCLK renamed /Display connector/DCLK
- net /DataEn renamed /Display connector/DataEn
- net /G0 renamed /Display connector/G0
- net /G1 renamed /Display connector/G1
- net /G2 renamed /Display connector/G2
- net /G3 renamed /Display connector/G3
- net /G4 renamed /Display connector/G4
- net /G5 renamed /Display connector/G5
- net /Hsync renamed /Display connector/Hsync
- net /R0 renamed /Display connector/R0
- net /R1 renamed /Display connector/R1
- net /R2 renamed /Display connector/R2
- net /R3 renamed /Display connector/R3
- net /R4 renamed /Display connector/R4
- net /R5 renamed /Display connector/R5
- net /Reset renamed /Display connector/Reset
- net /SCK renamed /Display connector/SCK
- net /SCS renamed /Display connector/SCS
- net /SDI renamed /Display connector/SDI
- net /Vsync renamed /Display connector/Vsync
- net /WC renamed /Display connector/WC
- C3 pad 1: Net-(C3-Pad1) -> +3V3
- C4 pad 1: Net-(C3-Pad1) -> +3V3
- J1 pad 1: +3V3 -> unconnected-(J1-3V3-Pad1)_1
- J1 pad 17: +3V3 -> unconnected-(J1-3V3-Pad1)
- L1 pad 2: Net-(C3-Pad1) -> +3V3
Routing:
- net /Display connector/R5: track 0.00 -> 122.3 mm, vias 0 -> 1
- net /Display connector/R0: track 0.00 -> 121.8 mm, vias 0 -> 1
- net /Display connector/R4: track 0.00 -> 121.2 mm, vias 0 -> 1
- net +5V: track 18.2 -> 138.1 mm
- net /Display connector/R3: track 0.00 -> 115.4 mm, vias 0 -> 1
- net /Display connector/G2: track 0.00 -> 111.8 mm, vias 0 -> 1
- net Net-(J1-GPIO24): track 0.00 -> 110.6 mm, vias 0 -> 1
- net /Display connector/G3: track 0.00 -> 107.4 mm, vias 0 -> 1
- net /Display connector/DCLK: track 0.00 -> 107.3 mm, vias 0 -> 1
- net /Display connector/B2: track 0.00 -> 102.6 mm, vias 0 -> 1
- net Net-(J1-GPIO23): track 0.00 -> 102.3 mm, vias 0 -> 1
- net /Display connector/B1: track 0.00 -> 101.8 mm, vias 0 -> 1
- net /Display connector/B3: track 0.00 -> 99.4 mm, vias 0 -> 1
- net /Display connector/DataEn: track 0.00 -> 99.3 mm, vias 0 -> 1
- net /Display connector/G1: track 0.00 -> 97.6 mm, vias 0 -> 1
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Other:
- outline, holes or cut-outs redrawn
- board text added: "B"
- board text added: "CLK"
- board text added: "G"
- board text added: "R"
- board text added: "Sync"
