File: pcb/pollin-lcd.kicad_pcb (KiCad board)
At the start: 2 copper layers, 2 parts, among them J1 Raspberry_Pi_2_3, J2 Conn_01x04_Pin

Commit message: connect display
Parts:
- removed J2: Conn_01x04_Pin, Connector_PinHeader_2.54mm:PinHeader_1x04_P2.54mm_Vertical_SMD_Pin1Right
- added C1: 10uF 6.3V, Capacitor_SMD:C_0805_2012Metric_Pad1.18x1.45mm_HandSolder, F.Cu at (78.8, 87.5)
- added C2: 1uF 16V, Capacitor_SMD:C_0603_1608Metric_Pad1.08x0.95mm_HandSolder, F.Cu at (83.3, 87.2)
- added C3: 100nF 50V, Capacitor_SMD:C_0805_2012Metric_Pad1.18x1.45mm_HandSolder, F.Cu at (78.8, 90.5)
- added C4: 10uF 6.3V, Capacitor_SMD:C_0805_2012Metric_Pad1.18x1.45mm_HandSolder, F.Cu at (78.8, 93.5)
- added C5: 10uF 6.3V, Capacitor_SMD:C_0805_2012Metric_Pad1.18x1.45mm_HandSolder, F.Cu at (170.5, 83.4)
- added C6: 100nF 50V, Capacitor_SMD:C_0805_2012Metric_Pad1.18x1.45mm_HandSolder, F.Cu at (174.0, 83.4)
- added C7: 100nF 50V, Capacitor_SMD:C_0805_2012Metric_Pad1.18x1.45mm_HandSolder, F.Cu at (170.5, 78.7)
- added J3: 505110-4091, Molex_505110-4091:5051104091, F.Cu at (155.5, 74.0)
- added L1: 2.2uH, Inductor_SMD:L_Bourns-SRN4018, F.Cu at (79.4, 83.2)
- added R1: 20k, Resistor_SMD:R_0603_1608Metric_Pad0.98x0.95mm_HandSolder, F.Cu at (83.3, 89.7)
- added R2: 100k, Resistor_SMD:R_0603_1608Metric_Pad0.98x0.95mm_HandSolder, F.Cu at (83.3, 92.2)
- added R3: 100k, Resistor_SMD:R_0603_1608Metric_Pad0.98x0.95mm_HandSolder, F.Cu at (83.3, 94.8)
- added R4: 10k, Resistor_SMD:R_0603_1608Metric_Pad0.98x0.95mm_HandSolder, F.Cu at (178.5, 85.4)
- added R5: 10k, Resistor_SMD:R_0603_1608Metric_Pad0.98x0.95mm_HandSolder, F.Cu at (181.5, 85.4)
- added REF**: Raspberry_Pi_Zero_Socketed_THT_FaceDown_MountingHoles, Module:Raspberry_Pi_Zero_Socketed_THT_FaceDown_MountingHoles, F.Cu at (51.2, 66.8)
- added U1: TLV62568DBV, Package_TO_SOT_SMD:SOT-23-5, F.Cu at (85.0, 82.8)
- J1: footprint Module:Raspberry_Pi_Zero_Socketed_THT_FaceDown_MountingHoles -> Connector_Samtec_HLE_SMD:Samtec_HLE-120-02-xxx-DV-BE-A_2x20_P2.54mm_Horizontal; moved to B.Cu
- moved J1 24.6 mm to (75.4, 68.0), turned to 180 degrees
Connections:
- J1 pad 10: Net-(J1-GPIO15/RXD) -> /G5
- J1 pad 11: unconnected-(J1-GPIO17-Pad11) -> /R1
- J1 pad 12: unconnected-(J1-GPIO18/PWM0-Pad12) -> /R2
- J1 pad 16: unconnected-(J1-GPIO23-Pad16) -> Net-(J1-GPIO23)
- J1 pad 18: unconnected-(J1-GPIO24-Pad18) -> Net-(J1-GPIO24)
- J1 pad 19: unconnected-(J1-MOSI0/GPIO10-Pad19) -> /G0
- J1 pad 21: unconnected-(J1-MISO0/GPIO9-Pad21) -> /B5
- J1 pad 23: unconnected-(J1-SCLK0/GPIO11-Pad23) -> /G1
- J1 pad 24: unconnected-(J1-~{CE0}/GPIO8-Pad24) -> /B4
- J1 pad 26: unconnected-(J1-~{CE1}/GPIO7-Pad26) -> /B3
- J1 pad 27: unconnected-(J1-ID_SD/GPIO0-Pad27) -> /DCLK
- J1 pad 28: unconnected-(J1-ID_SC/GPIO1-Pad28) -> /DataEn
- J1 pad 29: unconnected-(J1-GCLK1/GPIO5-Pad29) -> /B1
- J1 pad 3: unconnected-(J1-SDA/GPIO2-Pad3) -> /Vsync
- J1 pad 31: unconnected-(J1-GCLK2/GPIO6-Pad31) -> /B2
- J1 pad 32: unconnected-(J1-PWM0/GPIO12-Pad32) -> /G2
- J1 pad 33: unconnected-(J1-PWM1/GPIO13-Pad33) -> /G3
- J1 pad 35: unconnected-(J1-GPIO19/MISO1-Pad35) -> /R3
- J1 pad 36: unconnected-(J1-GPIO16-Pad36) -> /R0
- J1 pad 38: unconnected-(J1-GPIO20/MOSI1-Pad38) -> /R4
- J1 pad 40: unconnected-(J1-GPIO21/SCLK1-Pad40) -> /R5
- J1 pad 5: unconnected-(J1-SCL/GPIO3-Pad5) -> /Hsync
- J1 pad 7: unconnected-(J1-GCLK0/GPIO4-Pad7) -> /B0
- J1 pad 8: Net-(J1-GPIO14/TXD) -> /G4
Routing:
- net Net-(J1-GPIO15/RXD): track 36.0 -> 0.00 mm
- net Net-(J1-GPIO14/TXD): track 34.0 -> 0.00 mm
- net +3V3: track 0.00 -> 24.1 mm
- net +5V: track 23.1 -> 0.00 mm
- net /Reset: track 0.00 -> 11.8 mm
- added copper zone on B.Cu, net GND

Commit message: 🔥
Parts:
- added ?: , clipboard:8f9f653c-d1d4-44ae-8881-cd5268ffe7a2, F.Cu at (126.0, 0.00)
- Raspberry Pi Zero: renamed from REF**
- moved C7 56.8 mm to (144.6, 28.2)
- moved C5 56.8 mm to (144.6, 32.9)
- moved C6 56.8 mm to (148.1, 32.9)
- moved J3 56.8 mm to (129.6, 23.4)
- moved R4 56.8 mm to (152.6, 34.9)
- moved R5 56.8 mm to (155.6, 34.9)
- moved R2 52.0 mm to (67.0, 42.9), turned to 90 degrees
- moved C4 51.6 mm to (82.5, 42.0)
- moved R3 51.5 mm to (66.1, 46.2), turned to 180 degrees
- moved C1 48.1 mm to (71.0, 40.0), turned to 180 degrees
- moved Raspberry Pi Zero 47.6 mm to (22.1, 29.1)
- moved J1 46.5 mm to (48.0, 30.4)
- moved C3 44.6 mm to (82.5, 46.0)
- moved R1 44.0 mm to (66.1, 49.2), turned to 180 degrees
- moved U1 40.8 mm to (71.0, 44.5), turned to 180 degrees
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Routing:
- net +5V: track 0.00 -> 18.2 mm, vias 0 -> 3
- net Net-(U1-EN): track 0.00 -> 10.8 mm
- net Net-(C3-Pad1): track 0.00 -> 6.94 mm
- net Net-(U1-FB): track 0.00 -> 6.30 mm
- net Net-(U1-SW): track 0.00 -> 3.52 mm
Other:
- board outline added: 248 x 56 mm

Commit message: display connections done
Parts:
- added ?: , , F.Cu at (0.00, 31.5)
- added ?: , , F.Cu at (242.0, 34.1)
- moved R3 5.03 mm to (70.6, 48.5), turned to 0 degrees
- moved R1 0.76 mm to (66.0, 48.5)
- turned R4 to 90 degrees
- turned R5 to 90 degrees
Connections:
- net /B0 renamed /Display Connector/B0
- net /B1 renamed /Display Connector/B1
- net /B2 renamed /Display Connector/B2
- net /B3 renamed /Display Connector/B3
- net /B4 renamed /Display Connector/B4
- net /B5 renamed /Display Connector/B5
- net /DCLK renamed /Display Connector/DCLK
- net /DataEn renamed /Display Connector/DataEn
- net /G0 renamed /Display Connector/G0
- net /G1 renamed /Display Connector/G1
- net /G2 renamed /Display Connector/G2
- net /G3 renamed /Display Connector/G3
- net /G4 renamed /Display Connector/G4
- net /G5 renamed /Display Connector/G5
- net /Hsync renamed /Display Connector/Hsync
- net /R0 renamed /Display Connector/R0
- net /R1 renamed /Display Connector/R1
- net /R2 renamed /Display Connector/R2
- net /R3 renamed /Display Connector/R3
- net /R4 renamed /Display Connector/R4
- net /R5 renamed /Display Connector/R5
- net /Reset renamed /Display Connector/Reset
- net /SCK renamed /Display Connector/SCK
- net /SCS renamed /Display Connector/SCS
- net /SDI renamed /Display Connector/SDI
- net /Vsync renamed /Display Connector/Vsync
- net /WC renamed /Display Connector/WC
- C3 pad 1: Net-(C3-Pad1) -> +3V3
- C4 pad 1: Net-(C3-Pad1) -> +3V3
- J1 pad 1: +3V3 -> unconnected-(J1-3V3-Pad1)_1
- J1 pad 17: +3V3 -> unconnected-(J1-3V3-Pad1)
- L1 pad 2: Net-(C3-Pad1) -> +3V3
- R3 pad 2: unconnected-(R3-Pad2) -> +3V3
- R4 pad 1: +3V3 -> +5V
- R5 pad 1: +3V3 -> +5V
Routing:
- net /Display Connector/R5: track 0.00 -> 123.7 mm, vias 0 -> 1
- net /Display Connector/R0: track 0.00 -> 121.2 mm, vias 0 -> 1
- net /Display Connector/R4: track 0.00 -> 121.2 mm, vias 0 -> 1
- net /Display Connector/R3: track 0.00 -> 114.9 mm, vias 0 -> 1
- net +5V: track 18.2 -> 132.8 mm
- net /Display Connector/G2: track 0.00 -> 111.1 mm, vias 0 -> 1
- net /Display Connector/G3: track 0.00 -> 108.3 mm, vias 0 -> 1
- net /Display Connector/DCLK: track 0.00 -> 107.3 mm, vias 0 -> 1
- net /Display Connector/B2: track 0.00 -> 102.8 mm, vias 0 -> 1
- net /Display Connector/B1: track 0.00 -> 101.4 mm, vias 0 -> 1
- net /Display Connector/DataEn: track 0.00 -> 99.9 mm, vias 0 -> 1
- net /Display Connector/B3: track 0.00 -> 99.9 mm, vias 0 -> 1
- net /Display Connector/B4: track 0.00 -> 97.1 mm, vias 0 -> 1
- net /Display Connector/G1: track 0.00 -> 97.0 mm, vias 0 -> 1
- net /Display Connector/G0: track 0.00 -> 92.7 mm, vias 0 -> 1
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Other:
- outline, holes or cut-outs redrawn

Commit message: foo
Parts:
- removed ? (x2): , 
- removed ?: , clipboard:8f9f653c-d1d4-44ae-8881-cd5268ffe7a2
- moved R3 5.03 mm to (66.1, 46.2), turned to 180 degrees
- moved R1 0.76 mm to (66.1, 49.2)
- turned R4 to -90 degrees
- turned R5 to -90 degrees
Connections:
- net /Display Connector/B0 renamed /Display connector/B0
- net /Display Connector/B1 renamed /Display connector/B1
- net /Display Connector/B2 renamed /Display connector/B2
- net /Display Connector/B3 renamed /Display connector/B3
- net /Display Connector/B4 renamed /Display connector/B4
- net /Display Connector/B5 renamed /Display connector/B5
- net /Display Connector/DCLK renamed /Display connector/DCLK
- net /Display Connector/DataEn renamed /Display connector/DataEn
- net /Display Connector/G0 renamed /Display connector/G0
- net /Display Connector/G1 renamed /Display connector/G1
- net /Display Connector/G2 renamed /Display connector/G2
- net /Display Connector/G3 renamed /Display connector/G3
- net /Display Connector/G4 renamed /Display connector/G4
- net /Display Connector/G5 renamed /Display connector/G5
- net /Display Connector/Hsync renamed /Display connector/Hsync
- net /Display Connector/R0 renamed /Display connector/R0
- net /Display Connector/R1 renamed /Display connector/R1
- net /Display Connector/R2 renamed /Display connector/R2
- net /Display Connector/R3 renamed /Display connector/R3
- net /Display Connector/R4 renamed /Display connector/R4
- net /Display Connector/R5 renamed /Display connector/R5
- net /Display Connector/Reset renamed /Display connector/Reset
- net /Display Connector/SCK renamed /Display connector/SCK
- net /Display Connector/SCS renamed /Display connector/SCS
- net /Display Connector/SDI renamed /Display connector/SDI
- net /Display Connector/Vsync renamed /Display connector/Vsync
- net /Display Connector/WC renamed /Display connector/WC
- R3 pad 2: +3V3 -> unconnected-(R3-Pad2)
- R4 pad 1: +5V -> +3V3
- R5 pad 1: +5V -> +3V3
Routing:
- net Net-(J1-GPIO24): track 0.00 -> 110.6 mm, vias 0 -> 1
- net Net-(J1-GPIO23): track 0.00 -> 102.3 mm, vias 0 -> 1
- net +3V3: track 105.5 -> 88.0 mm, vias 6 -> 0
- net +5V: track 132.8 -> 138.1 mm
- net /Display connector/R2: track 90.0 -> 92.0 mm
- net /Display connector/R5: track 123.7 -> 122.3 mm
- net /Display connector/G4: track 80.2 -> 81.3 mm
- net /Display connector/Hsync: track 68.2 -> 69.2 mm
- net /Display connector/G3: track 108.3 -> 107.4 mm
- net /Display connector/G2: track 111.1 -> 111.8 mm
- net /Display connector/R0: track 121.2 -> 121.8 mm
- net /Display connector/DataEn: track 99.9 -> 99.3 mm
- net /Display connector/G1: track 97.0 -> 97.6 mm
- net (no net): vias 0 -> 3
Other:
- board text added: "B"
- board text added: "CLK"
- board text added: "G"
- board text added: "R"
- board text added: "Sync"
